File: rgbww-micro-board.kicad_pcb (KiCad board)
At the start: 2 copper layers, 44.5 x 33.8 mm, 39 parts, among them U1 dcdc-module, U2 ESP-12E

Commit message: add more gnd pads
Parts:
- added ?: GND, Connector_Wire:SolderWirePad_1x01_Drill0.8mm, F.Cu at (221.3, 79.8)
- added ?: GND, Connector_Wire:SolderWirePad_1x01_Drill0.8mm, F.Cu at (220.3, 60.9)
- added ?: GND, Connector_Wire:SolderWirePad_1x01_Drill0.8mm, F.Cu at (220.2, 58.2)
Routing:
- net GND: track 122.4 -> 125.3 mm
Changed lines of the file:
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@@
     (thickness 1.6)
     (drawings 9)
-    (tracks 224)
+    (tracks 226)
     (zones 0)
-    (modules 39)
+    (modules 42)
     (nets 24)
   )
@@
     (uvia_drill 0.1)
     (add_net +3V3)
+  )
+  (module Connector_Wire:SolderWirePad_1x01_Drill0.8mm (layer F.Cu)
+    (at 221.3 79.8)
+    (descr "Wire solder connection")
+    (tags connector)
+    (attr virtual)
+    (fp_text reference "" (at 0 -2.54) (layer F.SilkS)
+      (effects (font (size 1 1) (thickness 0.15)))
+    )
+    (fp_text value GND (at 2.7 -0.3) (layer F.Fab)
+      (effects (font (size 1 1) (thickness 0.15)))
+    )
+    (fp_text user %R (at 0 0) (layer F.Fab)
+      (effects (font (size 1 1) (thickness 0.15)))
+    )
+    (fp_line (start -1.5 -1.5) (end 1.5 -1.5) (layer F.CrtYd) (width 0.05))
+    (fp_line (start -1.5 -1.5) (end -1.5 1.5) (layer F.CrtYd) (width 0.05))
+    (fp_line (start 1.5 1.5) (end 1.5 -1.5) (layer F.CrtYd) (width 0.05))
+    (fp_line (start 1.5 1.5) (end -1.5 1.5) (layer F.CrtYd) (width 0.05))
+    (pad 1 thru_hole circle (at 0 0) (size 1.99898 1.99898) (drill 0.8001) (layers *.Cu *.Mask)
+      (net 2 GND))
+  )
+  (module Connector_Wire:SolderWirePad_1x01_Drill0.8mm (layer F.Cu)
+    (at 220.3 60.9)
+    (descr "Wire solder connection")
+    (tags connector)
+    (attr virtual)
+    (fp_text reference "" (at 0 -2.54) (layer F.SilkS)
+      (effects (font (size 1 1) (thickness 0.15)))
+    )
+    (fp_text value GND (at 0 2.54) (layer F.Fab)
+      (effects (font (size 1 1) (thickness 0.15)))
+    )
+    (fp_text user %R (at 0 0) (layer F.Fab)
+      (effects (font (size 1 1) (thickness 0.15)))
+    )
+    (fp_line (start -1.5 -1.5) (end 1.5 -1.5) (layer F.CrtYd) (width 0.05))
+    (fp_line (start -1.5 -1.5) (end -1.5 1.5) (layer F.CrtYd) (width 0.05))
+    (fp_line (start 1.5 1.5) (end 1.5 -1.5) (layer F.CrtYd) (width 0.05))
+    (fp_line (start 1.5 1.5) (end -1.5 1.5) (layer F.CrtYd) (width 0.05))
+    (pad 1 thru_hole circle (at 0 0) (size 1.99898 1.99898) (drill 0.8001) (layers *.Cu *.Mask)
+      (net 2 GND))
+  )
+  (module Connector_Wire:SolderWirePad_1x01_Drill0.8mm (layer F.Cu)
+    (at 220.2 58.2)
+    (descr "Wire solder connection")
+    (tags connector)
+    (attr virtual)
+    (fp_text reference "" (at 0 -2.54) (layer F.SilkS)
+      (effects (font (size 1 1) (thickness 0.15)))
+    )
+    (fp_text value GND (at 0 2.54) (layer F.Fab)
+      (effects (font (size 1 1) (thickness 0.15)))
+    )
+    (fp_line (start 1.5 1.5) (end -1.5 1.5) (layer F.CrtYd) (width 0.05))
+    (fp_line (start 1.5 1.5) (end 1.5 -1.5) (layer F.CrtYd) (width 0.05))
+    (fp_line (start -1.5 -1.5) (end -1.5 1.5) (layer F.CrtYd) (width 0.05))
+    (fp_line (start -1.5 -1.5) (end 1.5 -1.5) (layer F.CrtYd) (width 0.05))
+    (fp_text user %R (at 0 0) (layer F.Fab)
+      (effects (font (size 1 1) (thickness 0.15)))
+    )
+    (pad 1 thru_hole circle (at 0 0) (size 1.99898 1.99898) (drill 0.8001) (layers *.Cu *.Mask)
+      (net 2 GND))
   )
   (module Symbol:OSHW-Logo2_7.3x6mm_SilkScreen (layer B.Cu)
@@
     (descr "CP, Radial series, Radial, pin pitch=3.50mm, , diameter=10mm, Electrolytic Capacitor")
     (tags "CP Radial series Radial pin pitch 3.50mm  diameter 10mm Electrolytic Capacitor")
-    (fp_text reference C1 (at 2.5 -6.25) (layer F.SilkS)
+    (fp_text reference C1 (at 5.5 -4.9) (layer F.SilkS)
       (effects (font (size 1 1) (thickness 0.15)))
     )
@@
   (via (at 203.25 88.25) (size 0.8) (drill 0.4) (layers F.Cu B.Cu) (net 2))
   (via (at 204.5 86) (size 0.8) (drill 0.4) (layers F.Cu B.Cu) (net 2))
+  (segment (start 220.45 58.45) (end 220.2 58.2) (width 0.25) (layer F.Cu) (net 2))
+  (segment (start 223.05 58.45) (end 220.45 58.45) (width 0.25) (layer F.Cu) (net 2))
   (segment (start 232.5 82) (end 231.25 80.75) (width 0.7) (layer F.Cu) (net 3))
   (segment (start 232.5 87.75) (end 232.5 82) (width 0.7) (layer F.Cu) (net 3))
